File: PCB AND SCHEMATIC/compute model.kicad_pcb (KiCad board)
At the start: 4 copper layers, 87.1 x 154.9 mm, 100 parts, among them J1 260 SODIMM, J10 HDMI_A, J12 USB4115-03-C_REVA, J13 TOUCH, J14 solder pads for rf, J15 solder pads for wifi/bt, J2 Conn_02x11_Odd_Even, J5 Battery, J6 speaker 1, J7 speaker 1, U1 TLV75533PDQNR, U2 TS5A23157DGSR, U3 TPS61088RHLR, U4 AP2112K-1.8, U5 SSM2518CPZ, U6 BQ25895RTW, U7 USB2422/MJ, U8 BMI270, Y1 24MHZ

Commit message: Add files via upload
Routing:
- net (no net): track 21.2 -> 20.0 mm, vias 1 -> 0
- net CC2: track 138.8 -> 137.9 mm
- added copper zone on B.Cu, net GND
- added copper zone on In1.Cu, net GND
- added copper zone on In2.Cu, net GND
Changed lines of the file:
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@@
 	)
 	(segment
-		(start 139.182854 157.5)
-		(end 139.308064 157.62521)
-		(width 0.14986)
-		(layer "F.Cu")
-		(net 0)
-	)
-	(segment
-		(start 142.832854 158.8)
-		(end 141.758039 159.874815)
-		(width 0.14986)
-		(layer "F.Cu")
-		(net 0)
-	)
-	(segment
-		(start 141.758039 159.874815)
-		(end 140.705933 159.874815)
-		(width 0.14986)
-		(layer "F.Cu")
-		(net 0)
-	)
-	(segment
 		(start 137.682854 158.45)
 		(end 137.682854 157.485)
@@
 	)
 	(segment
-		(start 140.457083 159.630495)
-		(end 140.130495 159.630495)
-		(width 0.14986)
-		(layer "F.Cu")
-		(net 0)
-	)
-	(segment
 		(start 138.533761 158.8)
 		(end 138.032854 158.8)
@@
 	)
 	(segment
-		(start 140.705933 159.874815)
-		(end 140.457083 159.625965)
-		(width 0.14986)
-		(layer "F.Cu")
-		(net 0)
-	)
-	(segment
 		(start 143.5 154.5)
 		(end 144 155)
@@
 	)
 	(segment
-		(start 140.457083 159.625965)
-		(end 140.457083 159.630495)
-		(width 0.14986)
-		(layer "F.Cu")
-		(net 0)
-	)
-	(segment
 		(start 139.042087 158.291674)
 		(end 138.533761 158.8)
@@
 		(net 0)
 	)
-	(via
-		(at 140.130495 159.630495)
-		(size 0.40005)
-		(drill 0.100076)
-		(layers "F.Cu" "B.Cu")
-		(net 0)
-	)
-	(segment
-		(start 138.466946 159.537865)
-		(end 138.466946 159.234092)
-		(width 0.14986)
-		(layer "B.Cu")
-		(net 0)
-	)
 	(segment
-		(start 140.130495 159.630495)
-		(end 139.223946 159.630495)
-		(width 0.14986)
-		(layer "B.Cu")
-		(net 0)
-	)
-	(segment
-		(start 139.223946 159.630495)
-		(end 139.067726 159.786715)
-		(width 0.14986)
-		(layer "B.Cu")
-		(net 0)
-	)
-	(segment
-		(start 139.067726 159.786715)
-		(end 138.715796 159.786715)
-		(width 0.14986)
-		(layer "B.Cu")
+		(start 142.597508 158.564654)
+		(end 138.2682 158.564654)
+		(width 0.19812)
+		(layer "In2.Cu")
 		(net 0)
 	)
 	(segment
-		(start 138.466946 159.234092)
+		(start 138.2682 158.564654)
 		(end 138.032854 158.8)
-		(width 0.14986)
-		(layer "B.Cu")
+		(width 0.19812)
+		(layer "In2.Cu")
 		(net 0)
 	)
 	(segment
-		(start 138.715796 159.786715)
-		(end 138.466946 159.537865)
-		(width 0.14986)
-		(layer "B.Cu")
+		(start 142.832854 158.8)
+		(end 142.597508 158.564654)
+		(width 0.19812)
+		(layer "In2.Cu")
 		(net 0)
 	)
@@
 	)
 	(segment
-		(start 141.308064 158.13479)
-		(end 141.308064 157.61021)
+		(start 141.5 159.273785)
+		(end 141.43568 159.209465)
 		(width 0.14986)
 		(layer "F.Cu")
@@
 	)
 	(segment
-		(start 141.038822 159.45)
-		(end 140.881898 159.45)
-		(width 0.14986)
-		(layer "F.Cu")
-		(net 148)
-	)
-	(segment
 		(start 150 128.5)
 		(end 149.45 129.05)
@@
 	)
 	(segment
+		(start 141.43568 158.857535)
+		(end 141.5 158.793215)
+		(width 0.14986)
+		(layer "F.Cu")
+		(net 148)
+	)
+	(segment
 		(start 143 63.5)
 		(end 143 72.5)
@@
 	)
 	(segment
-		(start 141.43568 159.053142)
-		(end 141.038822 159.45)
-		(width 0.14986)
-		(layer "F.Cu")
-		(net 148)
-	)
-	(segment
 		(start 159.446101 138.0119)
 		(end 151 138.0119)
@@
 	)
 	(segment
-		(start 141.5 158.13479)
-		(end 141.308064 158.13479)
-		(width 0.14986)
-		(layer "F.Cu")
-		(net 148)
-	)
-	(segment
-		(start 141.43568 158.857535)
-		(end 141.43568 159.053142)
-		(width 0.14986)
-		(layer "F.Cu")
-		(net 148)
-	)
-	(segment
 		(start 147 106.45)
 		(end 147 110)
@@
 	)
 	(segment
+		(start 141.43568 159.209465)
+		(end 141.43568 158.857535)
+		(width 0.14986)
+		(layer "F.Cu")
+		(net 148)
+	)
+	(segment
 		(start 150.55 137.5619)
 		(end 151 138.0119)
@@
 	)
 	(segment
-		(start 149.45 129.05)
-		(end 149.45 137)
+		(start 141.308064 158.13479)
+		(end 141.308064 157.61021)
 		(width 0.14986)
 		(layer "F.Cu")
@@
 	)
 	(segment
-		(start 141.5 158.793215)
-		(end 141.43568 158.857535)
+		(start 141.5 158.13479)
+		(end 141.308064 158.13479)
+		(width 0.14986)
+		(layer "F.Cu")
+		(net 148)
+	)
+	(segment
+		(start 149.45 129.05)
+		(end 149.45 137)
 		(width 0.14986)
 		(layer "F.Cu")
@@
 	)
 	(segment
+		(start 141.5 159.45)
+		(end 141.5 159.273785)
+		(width 0.14986)
+		(layer "F.Cu")
+		(net 148)
+	)
+	(segment
 		(start 143 45.5)
 		(end 143 47.077679)
@@
 	)
 	(via
-		(at 140.881898 159.45)
+		(at 141.5 159.45)
 		(size 0.40005)
 		(drill 0.100076)
@@
 	)
 	(segment
-		(start 144 159.5)
-		(end 151.0381 152.4619)
+		(start 146.4754 105.9254)
+		(end 147 106.45)
 		(width 0.14986)
 		(layer "B.Cu")
@@
 	)
 	(segment
-		(start 146.4754 105.9254)
-		(end 147 106.45)
+		(start 151.0381 140.999515)
+		(end 151.018277 140.979692)
 		(width 0.14986)
 		(layer "B.Cu")
@@
 	)
 	(segment
-		(start 151.0381 140.999515)
-		(end 151.018277 140.979692)
+		(start 142.437135 159.5)
+		(end 142.511925 159.57479)
 		(width 0.14986)
 		(layer "B.Cu")
@@
 	)
 	(segment
+		(start 141.5 159.45)
+		(end 141.55 159.5)
+		(width 0.14986)
+		(layer "B.Cu")
+		(net 148)
+	)
+	(segment
 		(start 146.4754 73.803082)
 		(end 146.4754 105.9254)
@@
 	)
 	(segment
+		(start 142.511925 159.57479)
+		(end 143.153783 159.57479)
+		(width 0.14986)
+		(layer "B.Cu")
+		(net 148)
+	)
+	(segment
 		(start 143.400006 63.099994)
 		(end 143 63.5)
@@
 	)
 	(segment
-		(start 151.0381 152.4619)
-		(end 151.0381 140.999515)
+		(start 144 159.5)
+		(end 151.0381 152.4619)
 		(width 0.14986)
 		(layer "B.Cu")
@@
 	)
 	(segment
-		(start 143.228573 159.5)
-		(end 144 159.5)
-		(width 0.14986)
-		(layer "B.Cu")
-		(net 148)
-	)
-	(segment
 		(start 144 73.5)
 		(end 146.172318 73.5)
@@
 	)
 	(segment
-		(start 140.931898 159.5)
-		(end 142.437135 159.5)
-		(width 0.14986)
-		(layer "B.Cu")
-		(net 148)
-	)
-	(segment
-		(start 142.511925 159.57479)
-		(end 143.153783 159.57479)
+		(start 143.153783 159.57479)
+		(end 143.228573 159.5)
 		(width 0.14986)
 		(layer "B.Cu")
@@
 	)
 	(segment
-		(start 143.153783 159.57479)
-		(end 143.228573 159.5)
+		(start 149.45 137)
+		(end 150.05 137)
 		(width 0.14986)
 		(layer "B.Cu")
@@
 	)
 	(segment
-		(start 149.45 137)
-		(end 150.05 137)
+		(start 151.0381 152.4619)
+		(end 151.0381 140.999515)
 		(width 0.14986)
 		(layer "B.Cu")
@@
 	)
 	(segment
-		(start 142.437135 159.5)
-		(end 142.511925 159.57479)
+		(start 143.228573 159.5)
+		(end 144 159.5)
 		(width 0.14986)
 		(layer "B.Cu")
@@
 	)
 	(segment
-		(start 140.881898 159.45)
-		(end 140.931898 159.5)
+		(start 141.55 159.5)
+		(end 142.437135 159.5)
 		(width 0.14986)
 		(layer "B.Cu")
@@
 	)
 	(segment
-		(start 139.639094 157.5)
-		(end 137.5 157.5)
-		(width 0.14986)
-		(layer "B.Cu")
-		(net 174)
-	)
-	(segment
 		(start 140.5 51.375)
 		(end 140.5 45.194738)
@@
 	)
 	(segment
-		(start 137.5 157.5)
-		(end 135.5 159.5)
-		(width 0.14986)
-		(layer "B.Cu")
-		(net 174)
-	)
-	(segment
-		(start 140.163506 158.024412)
-		(end 139.639094 157.5)
-		(width 0.14986)
-		(layer "B.Cu")
-		(net 174)
-	)
-	(segment
 		(start 140.5 154.892331)
 		(end 140.5 153)
@@
 	)
 	(segment
+		(start 140.163506 158.024412)
+		(end 139.804918 157.665824)
+		(width 0.2)
+		(layer "In2.Cu")
+		(net 174)
+	)
+	(segment
+		(start 139.804918 157.665824)
+		(end 137.834176 157.665824)
+		(width 0.2)
+		(layer "In2.Cu")
+		(net 174)
+	)
+	(segment
+		(start 136 159.5)
+		(end 135.5 159.5)
+		(width 0.2)
+		(layer "In2.Cu")
+		(net 174)
+	)
+	(segment
+		(start 137.834176 157.665824)
+		(end 136 159.5)
+		(width 0.2)
+		(layer "In2.Cu")
+		(net 174)
+	)
+	(segment
 		(start 114.735609 95.7875)
 		(end 116.2875 95.7875)
@@
 			)
 		)
+	)
+	(zone
+		(net 2)
+		(net_name "GND")
+		(layers "F.Cu" "B.Cu" "In1.Cu" "In2.Cu")
+		(hatch edge 0.5)
+		(priority 2)
+		(connect_pads yes
+			(clearance 0.1524)
+		)
+		(min_thickness 0.1524)
+		(filled_areas_thickness no)
+		(fill yes
+			(thermal_gap 0.5)
+			(thermal_bridge_width 0.5)
+		)
+		(polygon
+			(pts
+				(xy 96.865709 5.547288) (xy 184 5.547288) (xy 184 160.452711) (xy 96.865709 160.452711)
+			)
+		)
